File: Hardware/ESC/Power.kicad_sch (KiCad schematic)
At the start: 32 parts, among them J1 BATT TERM, J24 PWR PROT, J25 PWR 3.3V, Q1 SI7220 NMOS, SW3 PWR, U2 LM2574HVM-3.3, U36 LTC4367

Commit message: ESC Rough Draft
Parts:
- removed C53: 10uF, Capacitor_SMD:C_1206_3216Metric, symbol Device:C_Small
- removed C53: 22uF, Capacitor_SMD:C_1206_3216Metric, symbol Device:C_Small
- removed C53: 220uF, Capacitor_SMD:C_1206_3216Metric, symbol Device:C_Small
- removed D44: 3.3VPWR, LED_SMD:LED_0603_1608Metric, symbol Device:LED_Small_Filled
- removed D44: PWR, LED_SMD:LED_0603_1608Metric, symbol Device:LED_Small_Filled
- removed TP5: VDC, symbol Connector:TestPoint
- added C53: 220uF, Capacitor_SMD:C_1206_3216Metric, symbol Device:C_Small
- added C53: 22uF, Capacitor_SMD:C_1206_3216Metric, symbol Device:C_Small
- added C53: 10uF, Capacitor_SMD:C_1206_3216Metric, symbol Device:C_Small
- added D44: 3.3VPWR, LED_SMD:LED_0603_1608Metric, symbol Device:LED_Small_Filled
- added D44: PWR, LED_SMD:LED_0603_1608Metric, symbol Device:LED_Small_Filled
- added TP5: GND, symbol Connector:TestPoint
- added TP5: VDC, symbol Connector:TestPoint
Connections:
- net +3.3V: now also C53.1
- net GND: now also C53.2, C53.2, C53.2, D44.1 (K), TP5.1
- net VBUS: now also C53.1, C53.1
- net VDC: now also D44.2 (A), TP5.1
- net at R84.2: now also D44.2 (A)
- net at R2.1: now also D44.1 (K)
