File: Hardware/Flight_Board/Flight_Board.kicad_sch (KiCad schematic)
At the start: 22 parts, among them J4 STLINK, SW1 STM_RST, SW2 BOOT, U1 STM32F446RETx, Y1 16MHz

Commit message: ESC Rough Draft
Parts:
- added TP3: nReset, TestPoint:TestPoint_Pad_D2.0mm, symbol Connector:TestPoint
- added TP7: Boot, TestPoint:TestPoint_Pad_D2.0mm, symbol Connector:TestPoint
Connections:
- net BOOT0: now also TP7.1
- net nRST: now also TP3.1
- net SDA: now reaches U1.59 (PB7)
- net SCL: now reaches U1.61 (PB8)
Other:
- added sheet Camera (Camera.kicad_sch)
- note added: "Physical bootloader"
- note added: "Physical reset"
Changed lines of the file:
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@@
   (junction (at 25.4 67.31) (diameter 0) (color 0 0 0 0)
   )
+  (junction (at 43.18 120.65) (diameter 0) (color 0 0 0 0)
+  )
   (junction (at 50.8 180.34) (diameter 0) (color 0 0 0 0)
   )
   (junction (at 27.94 160.02) (diameter 0) (color 0 0 0 0)
+  )
+  (junction (at 48.26 87.63) (diameter 0) (color 0 0 0 0)
   )
   (junction (at 86.36 156.21) (diameter 0) (color 0 0 0 0)
@@
     (stroke (width 0) (type default))
   )
+  (wire (pts (xy 48.26 90.17) (xy 48.26 87.63))
+    (stroke (width 0) (type default))
+  )
   (wire (pts (xy 115.57 182.88) (xy 115.57 189.23))
     (stroke (width 0) (type default))
@@
     (stroke (width 0) (type default))
   )
+  (wire (pts (xy 43.18 118.11) (xy 43.18 120.65))
+    (stroke (width 0) (type default))
+  )
   (wire (pts (xy 83.82 22.86) (xy 86.36 22.86))
     (stroke (width 0) (type default))
@@
     (stroke (width 0) (type default))
   )
+  (wire (pts (xy 50.8 87.63) (xy 48.26 87.63))
+    (stroke (width 0) (type default))
+  )
   (wire (pts (xy 25.4 66.04) (xy 25.4 67.31))
     (stroke (width 0) (type default))
@@
     (stroke (width 0) (type default))
   )
+  (wire (pts (xy 43.18 120.65) (xy 45.72 120.65))
+    (stroke (width 0) (type default))
+  )
   (wire (pts (xy 113.03 156.21) (xy 125.73 156.21))
     (stroke (width 0) (type default))
@@
     (stroke (width 0) (type default))
   )
+  (wire (pts (xy 48.26 87.63) (xy 45.72 87.63))
+    (stroke (width 0) (type default))
+  )
   (wire (pts (xy 48.26 44.45) (xy 48.26 55.88))
     (stroke (width 0) (type default))
@@
     (stroke (width 0) (type default))
   )
-  (wire (pts (xy 39.37 120.65) (xy 45.72 120.65))
+  (wire (pts (xy 39.37 120.65) (xy 43.18 120.65))
     (stroke (width 0) (type default))
   )
@@
   (text "MCU Decoupling\n" (at 81.28 146.05 0)
     (effects (font (size 2 2)) (justify left bottom))
+  )
+  (text "Physical reset\n\n" (at 35.56 113.03 0)
+    (effects (font (size 1.27 1.27)) (justify left bottom))
+  )
+  (text "Physical bootloader\n" (at 31.75 82.55 0)
+    (effects (font (size 1.27 1.27)) (justify left bottom))
   )
   (text "Decoupling capacitors for digital power connections.\n"
@@
     )
   )
-  (global_label "BOOT0" (shape input) (at 45.72 87.63 0) (fields_autoplaced)
+  (global_label "BOOT0" (shape input) (at 50.8 87.63 0) (fields_autoplaced)
     (effects (font (size 1.27 1.27)) (justify left))
-    (property "Intersheetrefs" "${INTERSHEET_REFS}" (at 54.8133 87.63 0)
+    (property "Intersheetrefs" "${INTERSHEET_REFS}" (at 59.8933 87.63 0)
       (effects (font (size 1.27 1.27)) (justify left) hide)
     )
@@
     (property "Intersheetrefs" "${INTERSHEET_REFS}" (at 21.2658 172.72 0)
       (effects (font (size 1.27 1.27)) (justify right) hide)
+    )
+  )
+  (global_label "SDA" (shape input) (at 106.68 92.71 0) (fields_autoplaced)
+    (effects (font (size 1.27 1.27)) (justify left))
+    (property "Intersheetrefs" "${INTERSHEET_REFS}" (at 113.2333 92.71 0)
+      (effects (font (size 1.27 1.27)) (justify left) hide)
+    )
+  )
+  (global_label "SCL" (shape input) (at 106.68 95.25 0) (fields_autoplaced)
+    (effects (font (size 1.27 1.27)) (justify left))
+    (property "Intersheetrefs" "${INTERSHEET_REFS}" (at 113.1728 95.25 0)
+      (effects (font (size 1.27 1.27)) (justify left) hide)
     )
   )
@@
     )
   )
+  (symbol (lib_id "Connector:TestPoint") (at 48.26 90.17 180) (unit 1)
+    (in_bom yes) (on_board yes) (dnp no) (fields_autoplaced)
+    (property "Reference" "TP7" (at 50.8 92.202 0)
+      (effects (font (size 1.27 1.27)) (justify right))
+    )
+    (property "Value" "Boot" (at 50.8 94.742 0)
+      (effects (font (size 1.27 1.27)) (justify right))
+    )
+    (property "Footprint" "TestPoint:TestPoint_Pad_D2.0mm" (at 43.18 90.17 0)
+      (effects (font (size 1.27 1.27)) hide)
+    )
+    (property "Datasheet" "~" (at 43.18 90.17 0)
+      (effects (font (size 1.27 1.27)) hide)
+    )
+    (pin "1")
+    (instances
+      (project "Flight_Board"
+        (path "/9bcc2c41-99de-46c1-94bb-5baa5251c91c"
+          (reference "TP7") (unit 1)
+        )
+      )
+    )
+  )
   (symbol (lib_id "Device:C") (at 139.7 160.02 0) (unit 1)
     (in_bom yes) (on_board yes) (dnp no) (fields_autoplaced)
@@
     )
   )
+  (symbol (lib_id "Connector:TestPoint") (at 43.18 118.11 0) (unit 1)
+    (in_bom yes) (on_board yes) (dnp no) (fields_autoplaced)
+    (property "Reference" "TP3" (at 45.72 113.538 0)
+      (effects (font (size 1.27 1.27)) (justify left))
+    )
+    (property "Value" "nReset" (at 45.72 116.078 0)
+      (effects (font (size 1.27 1.27)) (justify left))
+    )
+    (property "Footprint" "TestPoint:TestPoint_Pad_D2.0mm" (at 48.26 118.11 0)
+      (effects (font (size 1.27 1.27)) hide)
+    )
+    (property "Datasheet" "~" (at 48.26 118.11 0)
+      (effects (font (size 1.27 1.27)) hide)
+    )
+    (pin "1")
+    (instances
+      (project "Flight_Board"
+        (path "/9bcc2c41-99de-46c1-94bb-5baa5251c91c"
+          (reference "TP3") (unit 1)
+        )
+      )
+    )
+  )
   (symbol (lib_id "Device:R") (at 41.91 87.63 90) (unit 1)
     (in_bom yes) (on_board yes) (dnp no)
@@
     )
   )
-  (sheet (at 247.65 19.05) (size 31.75 31.75) (fields_autoplaced)
+  (sheet (at 245.11 19.05) (size 33.02 31.75) (fields_autoplaced)
     (stroke (width 0.1524) (type solid))
     (fill (color 0 0 0 0.0000))
-    (property "Sheetname" "Comms" (at 247.65 18.3384 0)
+    (property "Sheetname" "Comms" (at 245.11 18.3384 0)
       (effects (font (size 1.27 1.27)) (justify left bottom))
     )
-    (property "Sheetfile" "Comms.kicad_sch" (at 247.65 51.3846 0)
+    (property "Sheetfile" "Comms.kicad_sch" (at 245.11 51.3846 0)
       (effects (font (size 1.27 1.27)) (justify left top))
     )
@@
     )
   )
-  (sheet (at 205.74 19.05) (size 33.02 30.48) (fields_autoplaced)
+  (sheet (at 200.66 19.05) (size 33.02 30.48) (fields_autoplaced)
     (stroke (width 0.1524) (type solid))
     (fill (color 0 0 0 0.0000))
-    (property "Sheetname" "ESC" (at 205.74 18.3384 0)
+    (property "Sheetname" "ESC" (at 200.66 18.3384 0)
       (effects (font (size 1.27 1.27)) (justify left bottom))
     )
-    (property "Sheetfile" "ESC.kicad_sch" (at 205.74 50.1146 0)
+    (property "Sheetfile" "ESC.kicad_sch" (at 200.66 50.1146 0)
       (effects (font (size 1.27 1.27)) (justify left top))
     )
@@
       )
     )
+  )
+  (sheet (at 199.39 66.04) (size 34.29 33.02) (fields_autoplaced)
+    (stroke (width 0.1524) (type solid))
+    (fill (color 0 0 0 0.0000))
+    (property "Sheetname" "Camera" (at 199.39 65.3284 0)
+      (effects (font (size 1.27 1.27)) (justify left bottom))
+    )
+    (property "Sheetfile" "Camera.kicad_sch" (at 199.39 99.6446 0)
+      (effects (font (size 1.27 1.27)) (justify left top))
+    )
+    (instances
+      (project "Flight_Board"
+        (path "/9bcc2c41-99de-46c1-94bb-5baa5251c91c" (page "6"))
+      )
+    )
